File: mechanical_hardware/schematics/schematics.kicad_sch (KiCad schematic)
At the start: 0 parts

Commit message: kicad schematics
Parts:
- added BT1, BT2: Battery, symbol Device:Battery
- added F1: Fuse, symbol Device:Fuse
- added SW1: SW_Push, symbol Switch:SW_Push
- added U1, U2: IA2412D, Converter_DCDC:Converter_DCDC_XP_POWER-IAxxxxD_THT, symbol Converter_DCDC:IA2412D
- added U3: MPU-9250, Sensor_Motion:InvenSense_QFN-24_3x3mm_P0.4mm, symbol Sensor_Motion:MPU-9250
Connections:
- new net: BT1.1 (+), BT2.1 (+), F1.1
- new net: BT1.2 (-), BT2.2 (-)
- new net: F1.2, SW1.1
Other:
- note added: "COMMON GND bus"
- note added: "VBAT 7.4 V bus"
