File: mechanical_hardware/schematics/.history/schematics.kicad_sch (KiCad schematic)
At the start: 2 parts

Commit message: kicad schematics
Parts:
- added F1: Fuse, symbol Device:Fuse
- added SW1: SW_Push, symbol Switch:SW_Push
- added U1, U2: IA2412D, Converter_DCDC:Converter_DCDC_XP_POWER-IAxxxxD_THT, symbol Converter_DCDC:IA2412D
- added U3: MPU-9250, Sensor_Motion:InvenSense_QFN-24_3x3mm_P0.4mm, symbol Sensor_Motion:MPU-9250
Connections:
- net at BT1.1 (+): now also BT2.1 (+), F1.1
- net at BT1.2 (-): now also BT2.2 (-)
- new net: F1.2, SW1.1
Other:
- note added: "COMMON GND bus"
- note added: "VBAT 7.4 V bus"
- moved on the sheet: BT1, BT2

Commit message: cad
Parts:
- removed BT1, BT2: Battery, symbol Device:Battery
- removed F1: Fuse, symbol Device:Fuse
- removed SW1: SW_Push, symbol Switch:SW_Push
- removed U1, U2: IA2412D, Converter_DCDC:Converter_DCDC_XP_POWER-IAxxxxD_THT, symbol Converter_DCDC:IA2412D
- removed U3: MPU-9250, Sensor_Motion:InvenSense_QFN-24_3x3mm_P0.4mm, symbol Sensor_Motion:MPU-9250
- added BT1, BT2: Battery_Cell, symbol Device:Battery_Cell
- added U1:5,1V, U2:5V, U3:12V: CRE1S0305S3C, Converter_DCDC:Converter_DCDC_Murata_CRE1xxxxxx3C_THT, symbol Regulator_Switching:CRE1S0305S3C
Connections:
- new net: BT2.1 (+), U1:5,1V.2 (+VIN), U2:5V.2 (+VIN), U3:12V.2 (+VIN)
- new net: BT1.1 (+), BT2.2 (-)
- new net: BT1.2 (-), U1:5,1V.1 (-VIN), U2:5V.1 (-VIN), U3:12V.1 (-VIN)
Other:
- note removed: "COMMON GND bus"
- note removed: "VBAT 7.4 V bus"
