File: mechanical_hardware/schematics/.history/schematics.kicad_sch (KiCad schematic)
At the start: 5 parts, among them U1:5,1V CRE1S0305S3C, U2:5V CRE1S0305S3C, U3:12V CRE1S0305S3C

Commit message: schematics backup
Parts:
- removed U1:5,1V, U2:5V, U3:12V: CRE1S0305S3C, Converter_DCDC:Converter_DCDC_Murata_CRE1xxxxxx3C_THT, symbol Regulator_Switching:CRE1S0305S3C
- added JST1, JST2: Female, symbol Connector:Conn_01x02_Pin
- added JST3, JST4: Male, symbol Connector:Conn_01x02_Pin
- BT1, BT2: value Battery_Cell -> Battery_Cell 2000mAh
Connections:
- net at BT2.1 (+): now also JST2.2 (Pin_2)
- net at BT2.2 (-): now also JST2.1 (Pin_1); no longer BT1.1 (+)
- net at BT1.2 (-): now also JST1.1 (Pin_1)
- new net: BT1.1 (+), JST1.2 (Pin_2)
- new net: JST3.1 (Pin_1), JST4.2 (Pin_2)
Other:
- note added: "+"
- note added: "-"

Commit message: backup schematics
Parts:
- added J1: Raspberry_Pi_4, symbol Connector:Raspberry_Pi_4
- added M1, M2: N20 100RPM, symbol Motor:Motor_DC
- added MotorControl (x2): TB6612FNG, Package_SO:SSOP-24_5.3x8.2mm_P0.65mm, symbol Driver_Motor:TB6612FNG
- added SW1: PWR, symbol Switch:SW_SPST
- added U1: 5.1V - Pi, Converter_DCDC:Converter_DCDC_TRACO_TSR-1_THT, symbol Converter_DCDC:TSR_1-2412
- added U2: 5V ESP32, Converter_DCDC:Converter_DCDC_TRACO_TSR-1_THT, symbol Converter_DCDC:TSR_1-2412
- added U3: 11.5V motors, Converter_DCDC:Converter_DCDC_TRACO_TSR-1_THT, symbol Converter_DCDC:TSR_1-2412
- added U4: ESP32-C3, Package_DFN_QFN:QFN-32-1EP_5x5mm_P0.5mm_EP3.7x3.7mm, symbol MCU_Espressif:ESP32-C3
- added U5: MPU-9250, Sensor_Motion:InvenSense_QFN-24_3x3mm_P0.4mm, symbol Sensor_Motion:MPU-9250
Connections:
- net at BT2.1 (+): now also JST2.1 (Pin_1); no longer JST2.2 (Pin_2)
- net at BT2.2 (-): now also JST2.2 (Pin_2); no longer JST2.1 (Pin_1)
- net at JST1.1 (Pin_1): now also BT1.1 (+); no longer BT1.2 (-)
- net at JST1.2 (Pin_2): now also BT1.2 (-); no longer BT1.1 (+)
- net at JST3.2 (Pin_2): now also U1.2 (GND), U2.2 (GND), U3.2 (GND)
- net at JST4.1 (Pin_1): now also SW1.1 (A)
- new net: MotorControl.1 (AO1), MotorControl.2 (AO1) (x2)
- new net: MotorControl.10 (PGND2), MotorControl.9 (PGND2) (x2)
- new net: MotorControl.11 (BO1), MotorControl.12 (BO1) (x2)
- new net: MotorControl.3 (PGND1), MotorControl.4 (PGND1) (x2)
- new net: MotorControl.5 (AO2), MotorControl.6 (AO2) (x2)
- new net: MotorControl.7 (BO2), MotorControl.8 (BO2) (x2)
- new net: SW1.2 (B), U1.1 (Vin), U2.1 (Vin), U3.1 (Vin)
- new net: U4.2 (VDD3P3), U4.3 (VDD3P3)
- new net: U4.31 (VDDA), U4.32 (VDDA)
- new net: J1.1 (3V3), J1.17 (3V3)
- new net: J1.14 (GND), J1.20 (GND), J1.25 (GND), J1.30 (GND), J1.34 (GND), J1.39 (GND), J1.6 (GND), J1.9 (GND)
- new net: J1.2 (5V), J1.4 (5V)
Other:
- moved on the sheet: BT1, BT2, JST1, JST2, JST3, JST4
